File: OTlight.sch (KiCad schematic (older format))
At the start: 66 parts, among them P1 CONN_01X01, Q1 TEMT6000, Q2 RSR030N06TL, T1 TRANSFO, U1 LM3478, U10 IN-14, U11 IN-14, U12 MAX6931, U13 IN-14, U14 MAX6920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

Commit message: I2C footprint, silk and diode adjustments
Parts:
- removed P1: CONN_01X01, Connect:PINTST, symbol CONN_01X01
- added P1: CONN_01X02, Pin_Headers:Pin_Header_Straight_1x02_Pitch2.54mm, symbol CONN_01X02
Connections:
- wire segments 228 -> 229
Changed lines of the file:
@@
-$EndComp
-$Comp
-L CONN_01X01 P1
-U 1 1 58828AA9
-P 6150 1050
-F 0 "P1" H 6150 1150 50  0000 C CNN
-F 1 "CONN_01X01" V 6250 1050 50  0000 C CNN
-F 2 "Connect:PINTST" H 6150 1050 50  0001 C CNN
-F 3 "" H 6150 1050 50  0000 C CNN
-	1    6150 1050
-	1    0    0    -1
 $EndComp
 $Comp
@@
 Wire Wire Line
 	5350 6350 4300 6350
+$Comp
+L CONN_01X02 P1
+U 1 1 58E6E032
+P 6150 1100
+F 0 "P1" H 6150 1250 50  0000 C CNN
+F 1 "CONN_01X02" V 6250 1100 50  0000 C CNN
+F 2 "Pin_Headers:Pin_Header_Straight_1x02_Pitch2.54mm" H 6150 1100 50  0001 C CNN
+F 3 "" H 6150 1100 50  0000 C CNN
+	1    6150 1100
+	1    0    0    -1
+$EndComp
+$Comp
+L GND #PWR052
+U 1 1 58E6FDF3
+P 5950 1200
+F 0 "#PWR052" H 5950 950 50  0001 C CNN
+F 1 "GND" H 5950 1050 50  0000 C CNN
+F 2 "" H 5950 1200 50  0000 C CNN
+F 3 "" H 5950 1200 50  0000 C CNN
+	1    5950 1200
+	1    0    0    -1
+$EndComp
+Wire Wire Line
+	5950 1150 5950 1200
 $EndSCHEMATC

Commit message: Rev2 of the board Everything fits and is connected~
Parts:
- removed R24, R25, R26, R27, R28, R29, R30: R_Small, Resistors_SMD:R_0805_HandSoldering, symbol R_Small
- removed U10, U11, U13, U8: IN-14, BamboulabFootprints:IN-14, symbol IN-14
- removed U7: BME280, BamboulabFootprints:BME280-Angled, symbol BME280
- added C17: C_Small, Capacitors_SMD:C_0805_HandSoldering, symbol C_Small
- added C18: 0.1u, Capacitors_SMD:C_0805_HandSoldering, symbol C_Small
- added P2, P3, P4, P5: CONN_01X14, Pin_Headers:Pin_Header_Straight_2x07_Pitch1.27mm, symbol CONN_01X14
- added U7: bareBME280, BamboulabFootprints:BME280bare, symbol bareBME280
- U2: footprint BamboulabFootprints:NodeMCU-V3 -> BamboulabFootprints:NodeMCU-V2
- U3: footprint BamboulabFootprints:DS3231-Angled -> BamboulabFootprints:DS3231
Connections:
- net +3V3: now also R23.2, C18.2, U7.2 (CSB), U7.6 (VDDIO), U7.8 (VDD)
- net BLANK: no longer U12.13 (BLANK), U14.9 (BLANK), U2.20 (GPIO15), U9.13 (BLANK)
- net GND: now also D2.1 (K), U12.13 (BLANK), U14.9 (BLANK), U9.13 (BLANK), C17.1, C18.1, U7.1 (GND), U7.7 (GND)
- net HVout: now also P2.13 (P13), P3.13 (P13), P4.13 (P13), P5.13 (P13); no longer R17.1, R18.1, R19.1, R20.1
- net at U9.18 (OUT8): now also P2.9 (P9)
- net at U9.17 (OUT9): now also P2.10 (P10)
- net at U9.26 (OUT0): now also P2.1 (P1)
- net at R23.1: now also U7.5 (SDO)
- net at U9.25 (OUT1): now also P2.2 (P2)
- net at U9.24 (OUT2): now also P2.3 (P3)
- net at U9.23 (OUT3): now also P2.4 (P4)
- net at U9.22 (OUT4): now also P2.5 (P5)
- net at U9.21 (OUT5): now also P2.6 (P6)
- net at U9.20 (OUT6): now also P2.7 (P7)
- net at U9.19 (OUT7): now also P2.8 (P8)
- net at U12.26 (OUT0): now also P3.9 (P9)
- net at U12.25 (OUT1): now also P3.10 (P10)
- net at U9.10 (OUT12): now also P3.1 (P1)
- net at U9.9 (OUT13): now also P3.2 (P2)
- net at U9.8 (OUT14): now also P3.3 (P3)
- net at U9.7 (OUT15): now also P3.4 (P4)
- net at U9.6 (OUT16): now also P3.5 (P5)
- net at U9.5 (OUT17): now also P3.6 (P6)
- net at U9.4 (OUT18): now also P3.7 (P7)
- net at U9.3 (OUT19): now also P3.8 (P8)
- net at U12.10 (OUT12): now also P4.9 (P9)
- net at U12.9 (OUT13): now also P4.10 (P10)
- net at U12.22 (OUT4): now also P4.1 (P1)
- net at U12.21 (OUT5): now also P4.2 (P2)
- net at U12.20 (OUT6): now also P4.3 (P3)
- net at U12.19 (OUT7): now also P4.4 (P4)
- net at U12.18 (OUT8): now also P4.5 (P5)
- net at U12.17 (OUT9): now also P4.6 (P6)
- net at U12.12 (OUT10): now also P4.7 (P7)
- net at U12.11 (OUT11): now also P4.8 (P8)
- net at U14.14 (OUT4): now also P5.9 (P9)
- net at U14.13 (OUT5): now also P5.10 (P10)
- net at U12.6 (OUT16): now also P5.1 (P1)
- net at U12.5 (OUT17): now also P5.2 (P2)
- net at U12.4 (OUT18): now also P5.3 (P3)
- net at U12.3 (OUT19): now also P5.4 (P4)
- net at U14.18 (OUT0): now also P5.5 (P5)
- net at U14.17 (OUT1): now also P5.6 (P6)
- net at U14.16 (OUT2): now also P5.7 (P7)
- net at U14.15 (OUT3): now also P5.8 (P8)
- net at C12.2, C13.2, D2.2 (A)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: now also R16.2, C17.2
- net at U9.11 (OUT11): now also P2.12 (P12)
- net at U9.12 (OUT10): now also P2.11 (P11); no longer R23.2
- net at U12.23 (OUT3): now also P3.12 (P12)
- net at U12.24 (OUT2): now also P3.11 (P11)
- net at U12.7 (OUT15): now also P4.12 (P12)
- net at U12.8 (OUT14): now also P4.11 (P11)
- net at R22.2, U2.26 (GPIO2), U3.4 (SCL): now also U7.4 (SCK)
- net at R21.2, U2.27 (GPIO0), U3.3 (SDA): now also U7.3 (SDI)
- net at C9.1, R12.1: now also U2.20 (GPIO15); no longer U2.28 (GPIO4)
- net at C8.1, R11.1: now also U2.28 (GPIO4); no longer U2.29 (GPIO5)
- net at C7.1, R10.1: now also U2.29 (GPIO5); no longer U2.30 (GPIO16)
- net at U14.7 (OUT7): now also P5.12 (P12)
- net at U14.8 (OUT6): now also P5.11 (P11)
Other:
- moved on the sheet: D2, R17, R18, R19, R20

Commit message: Cleanup started
Parts:
- removed C11: 1u, Capacitors_SMD:C_2220_HandSoldering, symbol C_Small
Changed lines of the file:
@@
-$EndComp
-$Comp
-L C_Small C11
-U 1 1 586A7ABB
-P 5750 4350
-F 0 "C11" H 5760 4420 50  0000 L CNN
-F 1 "1u" H 5760 4270 50  0000 L CNN
-F 2 "Capacitors_SMD:C_2220_HandSoldering" H 5750 4350 50  0001 C CNN
-F 3 "" H 5750 4350 50  0000 C CNN
-	1    5750 4350
-	1    0    0    -1
 $EndComp
 $Comp
