File: _saved_OTlight.sch (KiCad schematic (older format))
At the start: 60 parts, among them P1 CONN_01X02, Q1 TEMT6000, Q2 RSR030N06TL, T1 TRANSFO, U1 LM3478, U10 IN-14, U11 IN-14, U12 MAX6931, U13 IN-14, U14 MAX6920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

Commit message: The start of bearing upgrade
Parts:
- U10, U11, U13, U8: footprint (none) -> BamboulabFootprints:IN-14-bearing-7mm
Changed lines of the file:
@@
 F 0 "U8" H 8800 2200 60  0000 C CNN
 F 1 "IN-14" H 8000 2200 60  0000 C CNN
-F 2 "" V 8650 1800 60  0001 C CNN
+F 2 "BamboulabFootprints:IN-14-bearing-7mm" V 8650 1800 60  0001 C CNN
 F 3 "" V 8650 1800 60  0001 C CNN
 	1    8350 1850
@@
 F 0 "U10" H 10450 2200 60  0000 C CNN
 F 1 "IN-14" H 9650 2200 60  0000 C CNN
-F 2 "" V 10300 1800 60  0001 C CNN
+F 2 "BamboulabFootprints:IN-14-bearing-7mm" V 10300 1800 60  0001 C CNN
 F 3 "" V 10300 1800 60  0001 C CNN
 	1    10000 1850
@@
 F 0 "U11" H 12100 2200 60  0000 C CNN
 F 1 "IN-14" H 11300 2200 60  0000 C CNN
-F 2 "" V 11950 1800 60  0001 C CNN
+F 2 "BamboulabFootprints:IN-14-bearing-7mm" V 11950 1800 60  0001 C CNN
 F 3 "" V 11950 1800 60  0001 C CNN
 	1    11650 1850
@@
 F 0 "U13" H 13750 2200 60  0000 C CNN
 F 1 "IN-14" H 12950 2200 60  0000 C CNN
-F 2 "" V 13600 1800 60  0001 C CNN
+F 2 "BamboulabFootprints:IN-14-bearing-7mm" V 13600 1800 60  0001 C CNN
 F 3 "" V 13600 1800 60  0001 C CNN
 	1    13300 1850
